File: pcb_TCA9548A/project.kicad_pcb (KiCad board)
At the start: 2 copper layers, 18.3 x 25.9 mm, 38 parts, among them IC1 TCA9548APWR

Commit message: Add panelize
Parts:
- added REF**: Tab, kikit:Tab, F.Cu at (141.7, 52.8)
- added REF**: Tab, kikit:Tab, F.Cu at (126.0, 79.3)
- added REF**: Tab, kikit:Tab, F.Cu at (126.0, 52.8)
- added REF**: Tab, kikit:Tab, F.Cu at (141.7, 79.3)

Commit message: Add revision number to PCB
Other:
- board text added: "Rev.: ${REVISION}"
