File: pcb_TCA9548A/project.kicad_sch (KiCad schematic)
At the start: 37 parts, among them IC1 TCA9548APWR

Commit message: Add revision number to PCB
Other:
- company: (none) -> Thomas Fanninger
- title: (none) -> Breakout Board: I²C Multiplexer based on TCA9548A
Changed lines of the file:
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@@
 	(generator_version "8.0")
 	(paper "A4")
+	(title_block
+		(title "Breakout Board: I²C Multiplexer based on TCA9548A")
+		(date "2024-06-09")
+		(rev "1")
+		(company "Thomas Fanninger")
+	)
 	(junction
 		(at 45.72 97.79)
